File: hardware/board/zmod4410.brd (EAGLE design)
At the start: 17.8 x 25.4 mm, 17 parts, among them IC1 ZMOD4410AI1R, Q2 BSS138, U2 AP2112K-3.3

Commit message: Modification to package
Parts:
- moved FID4 67.8 mm to (5.23, 20.9)
Changed lines of the file:
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@@
 </layers>
 <board>
-<fusionsync huburn="a.YnVzaW5lc3M6YW5zYWJpbzU" projecturn="a.YnVzaW5lc3M6YW5zYWJpbzUjMjAyMzAyMDg2MDcwOTUxNTY" f3durn="urn:adsk.wipprod:dm.lineage:9V34FLrOSAW0bTxlgEe4DQ" pcbguid="" lastpulledtime="2023-05-15T00:32:20Z" lastsyncedchangeguid="" latestrevisionid="0a70cbd3-452e-4b0b-a119-1680ff709b3d" lastsyncedrevisionid="0a70cbd3-452e-4b0b-a119-1680ff709b3d" lastboardhashguid="" lastpushedtime="" linktopcb3d="true"/>
+<fusionsync huburn="a.YnVzaW5lc3M6YW5zYWJpbzU" projecturn="a.YnVzaW5lc3M6YW5zYWJpbzUjMjAyMzAyMDg2MDcwOTUxNTY" f3durn="urn:adsk.wipprod:dm.lineage:7bTmPjb9TDGiVGh7-zgFZA" pcbguid="" lastpulledtime="" lastsyncedchangeguid="" latestrevisionid="d09e7211-b45a-483b-bd94-b7cec6f78d7f" lastsyncedrevisionid="d09e7211-b45a-483b-bd94-b7cec6f78d7f" lastboardhashguid="1caca547-48d5-8c8b-d8bf-b39afaa25965" lastpushedtime="2023-05-15T07:53:16Z" linktopcb3d="true"/>
 <plain>
 <wire x1="18.0966" y1="2.694" x2="18.0966" y2="23.014" width="0" layer="20" locked="yes"/>
@@
 <attribute name="MOUSER_PRICE-STOCK" value="https://www.mouser.com/Search/Refine.aspx?Keyword=964-ZMOD4410AI1R" x="13.97" y="34.29" size="1.778" layer="27" rot="R90" display="off"/>
 </element>
-<element name="J1" library="SparkFun-Connectors" library_urn="urn:adsk.eagle:library:2652347" package="1X04_1MM_RA" package3d_urn="urn:adsk.eagle:package:2652537/1" override_package3d_urn="urn:adsk.eagle:package:40382641/2" override_package_urn="urn:adsk.eagle:footprint:37714/1" value="" x="9.652" y="5.334" smashed="yes">
+<element name="J1" library="SparkFun-Connectors" library_urn="urn:adsk.eagle:library:2652347" package="1X04_1MM_RA" package3d_urn="urn:adsk.eagle:package:2652537/1" override_package3d_urn="urn:adsk.eagle:package:40382641/3" override_package_urn="urn:adsk.eagle:footprint:37714/1" value="" x="9.652" y="5.334" smashed="yes">
 <attribute name="PROD_ID" value="CONN-13694" x="26.162" y="-6.096" size="1.778" layer="27" display="off"/>
 <attribute name="VALUE" x="8.001" y="2.032" size="0.6096" layer="27" font="vector" ratio="20"/>
@@
 <attribute name="BOM" value="EXCLUDE" x="12.2428" y="18.9992" size="1.778" layer="27" display="off"/>
 </element>
-<element name="FID4" library="microbuilder" package="FIDUCIAL_1MM" value="FIDUCIAL_1MM" x="-30.48" y="-36.83" smashed="yes">
-<attribute name="BOM" value="EXCLUDE" x="-30.48" y="-39.37" size="1.778" layer="27" display="off"/>
+<element name="FID4" library="microbuilder" package="FIDUCIAL_1MM" value="FIDUCIAL_1MM" x="5.2324" y="20.8534" smashed="yes">
+<attribute name="BOM" value="EXCLUDE" x="5.2324" y="18.3134" size="1.778" layer="27" display="off"/>
 </element>
 </elements>
